File: gomagottcha/gomagottcha.sch (KiCad schematic (older format))
At the start: 87 parts, among them J1 USB_B_Micro, J2 Arduino_ICSP, SW1 SW_DIP_x01, U1 BM71BLES1FC2, U10 VMotor1670-1000-ND, U11 MOSNP, U12 VMotor1670-1000-ND, U13 Buzzer_490-9647-1-ND, U14 IMU, U2 FT232RL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

Commit message: changed all 100nF caps to 0.1uF
Parts:
- C28, C29, C31: value 100nF -> 0.1uF
Changed lines of the file:
@@
 P 13200 9600
 F 0 "C31" V 12948 9600 50  0000 C CNN
-F 1 "100nF" V 13350 9600 50  0000 C CNN
+F 1 "0.1uF" V 13350 9600 50  0000 C CNN
 F 2 "tama-footprints:C_0603_1608Metric" H 13238 9450 50  0001 C CNN
 F 3 "~" H 13200 9600 50  0001 C CNN
@@
 P 10950 9450
 F 0 "C28" V 10698 9450 50  0000 C CNN
-F 1 "100nF" V 10789 9450 50  0000 C CNN
+F 1 "0.1uF" V 10789 9450 50  0000 C CNN
 F 2 "tama-footprints:C_0603_1608Metric" H 10988 9300 50  0001 C CNN
 F 3 "~" H 10950 9450 50  0001 C CNN
@@
 P 13200 9050
 F 0 "C29" V 12948 9050 50  0000 C CNN
-F 1 "100nF" V 13039 9050 50  0000 C CNN
+F 1 "0.1uF" V 13039 9050 50  0000 C CNN
 F 2 "tama-footprints:C_0603_1608Metric" H 13238 8900 50  0001 C CNN
 F 3 "~" H 13200 9050 50  0001 C CNN
